File: SWAN_Client_Rev0/szakdolgozat.kicad_pcb (KiCad board)
At the start: 2 copper layers, 100 x 100 mm, 67 parts, among them J1 Barrel_Jack, J2 Conn_01x10_Female, J3 Conn_01x04_Female, J4 Conn_01x03_Female, K1 DIPxx-2Axx-21x, Q1 Q_PMOS_DGS, Q2 Q_NPN_BCE, SW1 SW_Push, SW2 SW_Push, U1 MCP1826S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

Commit message: Reference voltage for AWG is fixed
Parts:
- removed G***: LOGO, mylib:swan_logo
- R4: value 10k -> 100k
Connections:
- U3 pad 3: GND -> /1V65_REF
- U4 pad 4: GND -> /1V65_REF
- U7 pad 11: (no net) -> /1V65_REF
Routing:
- net /1V65_REF: track 0.00 -> 31.1 mm, vias 0 -> 3
- net GND: track 44.8 -> 41.4 mm, vias 32 -> 30
